File: Schematic/value_split/MCU - Power.kicad_sch (KiCad schematic)
At the start: 13 parts, among them U1 STM32G474RET3

Commit message: Update Outputs
Parts:
- C7: manf# 04023D475MAT2A -> CM05X5R475M25AH
Changed lines of the file:
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@@
       (effects (font (size 1.27 1.27)) (hide yes))
     )
-    (property "manf#" "04023D475MAT2A" (at 133.35 118.11 0)
+    (property "manf#" "CM05X5R475M25AH" (at 133.35 118.11 0)
       (effects (font (size 1.27 1.27)) (hide yes))
     )
