File: Schematic/value_split/User - LED Indicators.kicad_sch (KiCad schematic)
At the start: 10 parts, among them Q7 PMV90ENER, Q8 PMV90ENER

Commit message: Update Outputs
Parts:
- R26: manf# CRCW0402150RFKEDHP -> RCS0402150RFKED
Changed lines of the file:
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@@
       (effects (font (size 1.27 1.27)) (hide yes))
     )
-    (property "manf#" "CRCW0402150RFKEDHP" (at 198.12 67.31 0)
+    (property "manf#" "RCS0402150RFKED" (at 198.12 67.31 0)
       (effects (font (size 1.27 1.27)) (hide yes))
     )
