File: amulet_controller.kicad_sch (KiCad schematic)
At the start: 0 parts

Commit message: small changes
Other:
- note added: "${RELEASE_DATE_NUM}"
- note removed: "${CURRENT_DATE}"
Changed lines of the file:
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@@
 		)
 	)
-	(text "${CURRENT_DATE}"
+	(text "${RELEASE_DATE_NUM}"
 		(exclude_from_sim no)
 		(at 388.62 40.64 0)
