File: amulet_controller.kicad_sch (KiCad schematic)
At the start: 0 parts

Commit message: automatic ToC
Other:
- note added: "${SHEET_NAME_10}"
- note added: "${SHEET_NAME_11}"
- note added: "${SHEET_NAME_12}"
- note added: "${SHEET_NAME_13}"
- note added: "${SHEET_NAME_14}"
- note added: "${SHEET_NAME_15}"
- note added: "${SHEET_NAME_16}"
- note added: "${SHEET_NAME_17}"
- note added: "${SHEET_NAME_18}"
- note added: "${SHEET_NAME_19}"
- note added: "${SHEET_NAME_1}"
- note added: "${SHEET_NAME_20}"
- note added: "${SHEET_NAME_21}"
- note added: "${SHEET_NAME_22}"
- note added: "${SHEET_NAME_23}"
- note added: "${SHEET_NAME_24}"
- note added: "${SHEET_NAME_25}"
- note added: "${SHEET_NAME_26}"
- note added: "${SHEET_NAME_27}"
- note added: "${SHEET_NAME_28}"
- note added: "${SHEET_NAME_29}"
- note added: "${SHEET_NAME_2}"
- note added: "${SHEET_NAME_30}"
- note added: "${SHEET_NAME_31}"
- note added: "${SHEET_NAME_32}"
- note added: "${SHEET_NAME_33}"
- note added: "${SHEET_NAME_34}"
- note added: "${SHEET_NAME_35}"
- note added: "${SHEET_NAME_36}"
- note added: "${SHEET_NAME_37}"
- note added: "${SHEET_NAME_38}"
- note added: "${SHEET_NAME_39}"
- note added: "${SHEET_NAME_3}"
- note added: "${SHEET_NAME_40}"
- note added: "${SHEET_NAME_4}"
- note added: "${SHEET_NAME_5}"
- note added: "${SHEET_NAME_6}"
- note added: "${SHEET_NAME_7}"
- note added: "${SHEET_NAME_8}"
- note added: "${SHEET_NAME_9}"
- note removed: "..........................................."
- note removed: "Block Diagram"
- note removed: "Cover Page"
- note removed: "Interface - FD-CAN"
- note removed: "Interface - Fan Control"
- note removed: "Interface - Interconnects"
- note removed: "Interface - RS-422"
- note removed: "MCU - I/Os"
- note removed: "MCU - Power"
- note removed: "Misc - Board Version, DAC"
- note removed: "Misc - Holes, Fiducials"
- note removed: "Motor Control - Inverter"
- note removed: "Motor Control - Top Level"
- note removed: "Power - Connectors"
- note removed: "Power - Generation"
- note removed: "Power - Sequencing"
- note removed: "Project Architecture"
- note removed: "Revision History"
- note removed: "Sensing - Battery"
- note removed: "Sensing - Position"
- note removed: "Sensing - Temperature"
- note removed: "User - LED Indicators"
Changed lines of the file:
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@@
 		)
 	)
-	(text "..........................................."
+	(text "${SHEET_NAME_23}"
 		(exclude_from_sim no)
 		(at 243.84 99.06 0)
@@
 		)
 	)
-	(text "Misc - Board Version, DAC"
+	(text "${SHEET_NAME_10}"
 		(exclude_from_sim no)
 		(at 45.72 152.4 0)
@@
 		)
 	)
-	(text "Sensing - Battery"
+	(text "${SHEET_NAME_13}"
 		(exclude_from_sim no)
 		(at 144.78 99.06 0)
@@
 		)
 	)
-	(text "Interface - RS-422"
+	(text "${SHEET_NAME_15}"
 		(exclude_from_sim no)
 		(at 144.78 114.3 0)
@@
 		)
 	)
-	(text "Power - Connectors"
+	(text "${SHEET_NAME_7}"
 		(exclude_from_sim no)
 		(at 45.72 129.54 0)
@@
 		)
 	)
-	(text "..........................................."
+	(text "${SHEET_NAME_30}"
 		(exclude_from_sim no)
 		(at 243.84 152.4 0)
@@
 		)
 	)
-	(text "Interface - Interconnects"
+	(text "${SHEET_NAME_18}"
 		(exclude_from_sim no)
 		(at 144.78 137.16 0)
@@
 		)
 	)
-	(text "MCU - Power"
+	(text "${SHEET_NAME_4}"
 		(exclude_from_sim no)
 		(at 45.72 106.68 0)
@@
 		)
 	)
-	(text "..........................................."
+	(text "${SHEET_NAME_27}"
 		(exclude_from_sim no)
 		(at 243.84 129.54 0)
@@
 		)
 	)
-	(text "Power - Sequencing"
+	(text "${SHEET_NAME_20}"
 		(exclude_from_sim no)
 		(at 144.78 152.4 0)
@@
 		)
 	)
-	(text "..........................................."
+	(text "${SHEET_NAME_38}"
 		(exclude_from_sim no)
 		(at 342.9 137.16 0)
@@
 		)
 	)
-	(text "Motor Control - Inverter"
+	(text "${SHEET_NAME_9}"
 		(exclude_from_sim no)
 		(at 45.72 144.78 0)
@@
 		)
 	)
-	(text "Sensing - Temperature"
+	(text "${SHEET_NAME_12}"
 		(exclude_from_sim no)
 		(at 144.78 91.44 0)
@@
 		)
 	)
-	(text "..........................................."
+	(text "${SHEET_NAME_40}"
 		(exclude_from_sim no)
 		(at 342.9 152.4 0)
@@
 		)
 	)
-	(text "Misc - Holes, Fiducials"
+	(text "${SHEET_NAME_19}"
 		(exclude_from_sim no)
 		(at 144.78 144.78 0)
@@
 		)
 	)
-	(text "..........................................."
+	(text "${SHEET_NAME_32}"
 		(exclude_from_sim no)
 		(at 342.9 91.44 0)
@@
 		)
 	)
-	(text "User - LED Indicators"
+	(text "${SHEET_NAME_11}"
 		(exclude_from_sim no)
 		(at 144.78 83.82 0)
@@
 		)
 	)
-	(text "Motor Control - Top Level"
+	(text "${SHEET_NAME_8}"
 		(exclude_from_sim no)
 		(at 45.72 137.16 0)
@@
 		)
 	)
-	(text "..........................................."
+	(text "${SHEET_NAME_24}"
 		(exclude_from_sim no)
 		(at 243.84 106.68 0)
@@
 		)
 	)
-	(text "..........................................."
+	(text "${SHEET_NAME_29}"
 		(exclude_from_sim no)
 		(at 243.84 144.78 0)
@@
 		)
 	)
-	(text "..........................................."
+	(text "${SHEET_NAME_22}"
 		(exclude_from_sim no)
 		(at 243.84 91.44 0)
@@
 		)
 	)
-	(text "..........................................."
+	(text "${SHEET_NAME_39}"
 		(exclude_from_sim no)
 		(at 342.9 144.78 0)
@@
 		)
 	)
-	(text "MCU - I/Os"
+	(text "${SHEET_NAME_5}"
 		(exclude_from_sim no)
 		(at 45.72 114.3 0)
@@
 		)
 	)
-	(text "Interface - Fan Control"
+	(text "${SHEET_NAME_17}"
 		(exclude_from_sim no)
 		(at 144.78 129.54 0)
@@
 		)
 	)
-	(text "..........................................."
+	(text "${SHEET_NAME_28}"
 		(exclude_from_sim no)
 		(at 243.84 137.16 0)
@@
 		)
 	)
-	(text "..........................................."
+	(text "${SHEET_NAME_31}"
 		(exclude_from_sim no)
 		(at 342.9 83.82 0)
@@
 		)
 	)
-	(text "..........................................."
+	(text "${SHEET_NAME_26}"
 		(exclude_from_sim no)
 		(at 243.84 121.92 0)
@@
 		)
 	)
-	(text "..........................................."
+	(text "${SHEET_NAME_34}"
 		(exclude_from_sim no)
 		(at 342.9 106.68 0)
@@
 		)
 	)
-	(text "Power - Generation"
+	(text "${SHEET_NAME_6}"
 		(exclude_from_sim no)
 		(at 45.72 121.92 0)
@@
 		)
 	)
-	(text "Revision History"
+	(text "${SHEET_NAME_21}"
 		(exclude_from_sim no)
 		(at 243.84 83.82 0)
@@
 		)
 	)
-	(text "..........................................."
+	(text "${SHEET_NAME_36}"
 		(exclude_from_sim no)
 		(at 342.9 121.92 0)
@@
 		)
 	)
-	(text "..........................................."
+	(text "${SHEET_NAME_35}"
 		(exclude_from_sim no)
 		(at 342.9 114.3 0)
@@
 		)
 	)
-	(text "Block Diagram"
+	(text "${SHEET_NAME_2}"
 		(exclude_from_sim no)
 		(at 45.72 91.44 0)
@@
 		)
 	)
-	(text "Interface - FD-CAN"
+	(text "${SHEET_NAME_16}"
 		(exclude_from_sim no)
 		(at 144.78 121.92 0)
@@
 		)
 	)
-	(text "..........................................."
+	(text "${SHEET_NAME_25}"
 		(exclude_from_sim no)
 		(at 243.84 114.3 0)
@@
 		)
 	)
-	(text "..........................................."
+	(text "${SHEET_NAME_33}"
 		(exclude_from_sim no)
 		(at 342.9 99.06 0)
@@
 		)
 	)
-	(text "Cover Page"
+	(text "${SHEET_NAME_1}"
 		(exclude_from_sim no)
 		(at 45.72 83.82 0)
@@
 		)
 	)
-	(text "Sensing - Position"
+	(text "${SHEET_NAME_14}"
 		(exclude_from_sim no)
 		(at 144.78 106.68 0)
@@
 		)
 	)
-	(text "Project Architecture"
+	(text "${SHEET_NAME_3}"
 		(exclude_from_sim no)
 		(at 45.72 99.06 0)
@@
 		)
 	)
-	(text "..........................................."
+	(text "${SHEET_NAME_37}"
 		(exclude_from_sim no)
 		(at 342.9 129.54 0)
