File: Interface - FD-CAN.kicad_sch (KiCad schematic)
At the start: 4 parts, among them U10 TCAN1051HGVDRBRQ1

Commit message: Updated files without navigate_results
Parts:
- C108, C109: Manufacturer (none) -> Murata Electronics; Manufacturer Part Number (none) -> GCM155R71H104KE02J; manf Murata Electronics -> (none); manf# GCM155R71H104KE02J -> (none)
- R33: Manufacturer (none) -> YAGEO; Manufacturer Part Number (none) -> RT0402FRE0710KL; manf YAGEO -> (none); manf# RT0402FRE0710KL -> (none)
- U10: Manufacturer (none) -> Texas Instruments; Manufacturer Part Number (none) -> TCAN1051HGVDRBRQ1; manf Texas Instruments -> (none); manf# TCAN1051HGVDRBRQ1 -> (none)
Changed lines of the file:
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@@
 			)
 		)
-		(property "manf" "Texas Instruments"
+		(property "Manufacturer" "Texas Instruments"
 			(at 152.4 95.25 0)
 			(effects
@@
 			)
 		)
-		(property "manf#" "TCAN1051HGVDRBRQ1"
+		(property "Manufacturer Part Number" "TCAN1051HGVDRBRQ1"
 			(at 152.4 95.25 0)
 			(effects
@@
 			)
 		)
-		(property "manf" "Murata Electronics"
+		(property "Manufacturer" "Murata Electronics"
 			(at 170.18 73.66 0)
 			(effects
@@
 			)
 		)
-		(property "manf#" "GCM155R71H104KE02J"
+		(property "Manufacturer Part Number" "GCM155R71H104KE02J"
 			(at 170.18 73.66 0)
 			(effects
@@
 			)
 		)
-		(property "manf" "Murata Electronics"
+		(property "Manufacturer" "Murata Electronics"
 			(at 134.62 73.66 0)
 			(effects
@@
 			)
 		)
-		(property "manf#" "GCM155R71H104KE02J"
+		(property "Manufacturer Part Number" "GCM155R71H104KE02J"
 			(at 134.62 73.66 0)
 			(effects
@@
 			)
 		)
-		(property "manf" "YAGEO"
+		(property "Manufacturer" "YAGEO"
 			(at 129.54 105.41 0)
 			(effects
@@
 			)
 		)
-		(property "manf#" "RT0402FRE0710KL"
+		(property "Manufacturer Part Number" "RT0402FRE0710KL"
 			(at 129.54 105.41 0)
 			(effects
