File: Interface - Fan Control.kicad_sch (KiCad schematic)
At the start: 6 parts, among them Q9 PMV90ENER, U11 DGD0216WT-7

Commit message: Updated files without navigate_results
Parts:
- C110: Manufacturer (none) -> Murata Electronics; Manufacturer Part Number (none) -> GRM188Z71C475KE21J; manf Murata Electronics -> (none); manf# GRM188Z71C475KE21J -> (none)
- C111: Manufacturer (none) -> Murata Electronics; Manufacturer Part Number (none) -> GCM155R71H104KE02J; manf Murata Electronics -> (none); manf# GCM155R71H104KE02J -> (none)
- Q9: Manufacturer (none) -> Nexperia USA Inc.; Manufacturer Part Number (none) -> PMV90ENER; manf Nexperia USA Inc. -> (none); manf# PMV90ENER -> (none)
- R34: Manufacturer (none) -> Vishay; Manufacturer Part Number (none) -> CRCW060310R0FKEAHP; manf Vishay -> (none); manf# CRCW060310R0FKEAHP -> (none)
- U11: Manufacturer (none) -> Diodes Incorporated; Manufacturer Part Number (none) -> DGD0216WT-7; manf Diodes Incorporated -> (none); manf# DGD0216WT-7 -> (none)
Changed lines of the file:
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@@
 			)
 		)
-		(property "manf" "Murata Electronics"
+		(property "Manufacturer" "Murata Electronics"
 			(at 104.14 72.39 0)
 			(effects
@@
 			)
 		)
-		(property "manf#" "GRM188Z71C475KE21J"
+		(property "Manufacturer Part Number" "GRM188Z71C475KE21J"
 			(at 104.14 72.39 0)
 			(effects
@@
 			)
 		)
-		(property "manf" "Vishay"
+		(property "Manufacturer" "Vishay"
 			(at 160.02 91.44 0)
 			(effects
@@
 			)
 		)
-		(property "manf#" "CRCW060310R0FKEAHP"
+		(property "Manufacturer Part Number" "CRCW060310R0FKEAHP"
 			(at 160.02 91.44 0)
 			(effects
@@
 			)
 		)
-		(property "manf" "Diodes Incorporated"
+		(property "Manufacturer" "Diodes Incorporated"
 			(at 135.89 91.44 0)
 			(effects
@@
 			)
 		)
-		(property "manf#" "DGD0216WT-7"
+		(property "Manufacturer Part Number" "DGD0216WT-7"
 			(at 135.89 91.44 0)
 			(effects
@@
 			)
 		)
-		(property "manf" "Nexperia USA Inc."
+		(property "Manufacturer" "Nexperia USA Inc."
 			(at 179.07 91.44 0)
 			(effects
@@
 			)
 		)
-		(property "manf#" "PMV90ENER"
+		(property "Manufacturer Part Number" "PMV90ENER"
 			(at 179.07 91.44 0)
 			(effects
@@
 			)
 		)
-		(property "manf" "Murata Electronics"
+		(property "Manufacturer" "Murata Electronics"
 			(at 120.65 72.39 0)
 			(effects
@@
 			)
 		)
-		(property "manf#" "GCM155R71H104KE02J"
+		(property "Manufacturer Part Number" "GCM155R71H104KE02J"
 			(at 120.65 72.39 0)
 			(effects
