File: Interface - RS-422.kicad_sch (KiCad schematic)
At the start: 2 parts, among them U9 SN65HVD35DR

Commit message: Updated files without navigate_results
Parts:
- C107: Manufacturer (none) -> Murata Electronics; Manufacturer Part Number (none) -> GCM155R71H104KE02J; manf Murata Electronics -> (none); manf# GCM155R71H104KE02J -> (none)
- U9: Manufacturer (none) -> Texas Instruments; Manufacturer Part Number (none) -> SN65HVD35DR; manf Texas Instruments -> (none); manf# SN65HVD35DR -> (none)
Changed lines of the file:
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@@
 			)
 		)
-		(property "manf" "Murata Electronics"
+		(property "Manufacturer" "Murata Electronics"
 			(at 128.27 59.69 0)
 			(effects
@@
 			)
 		)
-		(property "manf#" "GCM155R71H104KE02J"
+		(property "Manufacturer Part Number" "GCM155R71H104KE02J"
 			(at 128.27 59.69 0)
 			(effects
@@
 			)
 		)
-		(property "manf" "Texas Instruments"
-			(at 146.05 85.09 0)
-			(effects
-				(font
-					(size 1.27 1.27)
-				)
-				(hide yes)
-			)
-		)
-		(property "manf#" "SN65HVD35DR"
-			(at 146.05 85.09 0)
-			(effects
+		(property "Manufacturer" "Texas Instruments"
+			(at 146.05 85.09 0)
+			(effects
+				(font
+					(size 1.27 1.27)
+				)
+				(hide yes)
+			)
+		)
+		(property "Manufacturer Part Number" "SN65HVD35DR"
+			(at 146.05 85.09 0)
+			(effects
