File: MCU - IOs.kicad_sch (KiCad schematic)
At the start: 45 parts, among them U1 STM32G474RET3

Commit message: Updated files without navigate_results
Parts:
- C12, C13, C14: Manufacturer (none) -> YAGEO; Manufacturer Part Number (none) -> AC0402KRX7R8BB102; manf YAGEO -> (none); manf# AC0402KRX7R8BB102 -> (none)
- R1, R2, R3: Manufacturer (none) -> Panasonic Electronic Components; Manufacturer Part Number (none) -> ERJ-2RKF22R0X; manf Panasonic Electronic Components -> (none); manf# ERJ-2RKF22R0X -> (none)
- U1: Manufacturer (none) -> STMicroelectronics; Manufacturer Part Number (none) -> STM32G474RET3; manf STMicroelectronics -> (none); manf# STM32G474RET3 -> (none)
Changed lines of the file:
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@@
 			)
 		)
-		(property "manf" "YAGEO"
+		(property "Manufacturer" "YAGEO"
 			(at 170.18 173.99 0)
 			(effects
@@
 			)
 		)
-		(property "manf#" "AC0402KRX7R8BB102"
+		(property "Manufacturer Part Number" "AC0402KRX7R8BB102"
 			(at 170.18 173.99 0)
 			(effects
@@
 			)
 		)
-		(property "manf" "Panasonic Electronic Components"
+		(property "Manufacturer" "Panasonic Electronic Components"
 			(at 185.42 165.1 0)
 			(effects
@@
 			)
 		)
-		(property "manf#" "ERJ-2RKF22R0X"
+		(property "Manufacturer Part Number" "ERJ-2RKF22R0X"
 			(at 185.42 165.1 0)
 			(effects
@@
 			)
 		)
-		(property "manf" "YAGEO"
+		(property "Manufacturer" "YAGEO"
 			(at 175.26 173.99 0)
 			(effects
@@
 			)
 		)
-		(property "manf#" "AC0402KRX7R8BB102"
+		(property "Manufacturer Part Number" "AC0402KRX7R8BB102"
 			(at 175.26 173.99 0)
 			(effects
@@
 			)
 		)
-		(property "manf" "Panasonic Electronic Components"
+		(property "Manufacturer" "Panasonic Electronic Components"
 			(at 185.42 167.64 0)
 			(effects
@@
 			)
 		)
-		(property "manf#" "ERJ-2RKF22R0X"
+		(property "Manufacturer Part Number" "ERJ-2RKF22R0X"
 			(at 185.42 167.64 0)
 			(effects
@@
 			)
 		)
-		(property "manf" "YAGEO"
+		(property "Manufacturer" "YAGEO"
 			(at 180.34 173.99 0)
 			(effects
@@
 			)
 		)
-		(property "manf#" "AC0402KRX7R8BB102"
+		(property "Manufacturer Part Number" "AC0402KRX7R8BB102"
 			(at 180.34 173.99 0)
 			(effects
@@
 			)
 		)
-		(property "manf" "STMicroelectronics"
+		(property "Manufacturer" "STMicroelectronics"
 			(at 88.9 91.44 0)
 			(effects
@@
 			)
 		)
-		(property "manf#" "STM32G474RET3"
+		(property "Manufacturer Part Number" "STM32G474RET3"
 			(at 88.9 91.44 0)
 			(effects
@@
 			)
 		)
-		(property "manf" "Panasonic Electronic Components"
+		(property "Manufacturer" "Panasonic Electronic Components"
 			(at 185.42 170.18 0)
 			(effects
@@
 			)
 		)
-		(property "manf#" "ERJ-2RKF22R0X"
+		(property "Manufacturer Part Number" "ERJ-2RKF22R0X"
 			(at 185.42 170.18 0)
 			(effects
