File: MCU - Power.kicad_sch (KiCad schematic)
At the start: 13 parts, among them U1 STM32G474RET3

Commit message: Updated files without navigate_results
Parts:
- C1: Manufacturer (none) -> Murata Electronics; Manufacturer Part Number (none) -> GRM188Z71C475KE21J; manf Murata Electronics -> (none); manf# GRM188Z71C475KE21J -> (none)
- C10, C11, C3, C4, C5, C8: Manufacturer (none) -> Murata Electronics; Manufacturer Part Number (none) -> GCM155R71H104KE02J; manf Murata Electronics -> (none); manf# GCM155R71H104KE02J -> (none)
- C2, C6, C9: Manufacturer (none) -> Murata Electronics; Manufacturer Part Number (none) -> GRM155Z71A105KE01J; manf Murata Electronics -> (none); manf# GRM155Z71A105KE01J -> (none)
- C7: Manufacturer (none) -> KYOCERA AVX; Manufacturer Part Number (none) -> CM05X5R475M25AH; manf KYOCERA AVX -> (none); manf# CM05X5R475M25AH -> (none)
- FB1: Manufacturer (none) -> Würth Elektronik; Manufacturer Part Number (none) -> 742792096; manf Würth Elektronik -> (none); manf# 742792096 -> (none)
- U1: Manufacturer (none) -> STMicroelectronics; Manufacturer Part Number (none) -> STM32G474RET3; manf STMicroelectronics -> (none); manf# STM32G474RET3 -> (none)
Changed lines of the file:
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@@
 			)
 		)
-		(property "manf" "Murata Electronics"
+		(property "Manufacturer" "Murata Electronics"
 			(at 105.41 77.47 0)
 			(effects
@@
 			)
 		)
-		(property "manf#" "GCM155R71H104KE02J"
+		(property "Manufacturer Part Number" "GCM155R71H104KE02J"
 			(at 105.41 77.47 0)
 			(effects
@@
 			)
 		)
-		(property "manf" "Murata Electronics"
+		(property "Manufacturer" "Murata Electronics"
 			(at 149.86 99.06 0)
 			(effects
@@
 			)
 		)
-		(property "manf#" "GCM155R71H104KE02J"
+		(property "Manufacturer Part Number" "GCM155R71H104KE02J"
 			(at 149.86 99.06 0)
 			(effects
@@
 			)
 		)
-		(property "manf" "Murata Electronics"
+		(property "Manufacturer" "Murata Electronics"
 			(at 133.35 77.47 0)
 			(effects
@@
 			)
 		)
-		(property "manf#" "GCM155R71H104KE02J"
+		(property "Manufacturer Part Number" "GCM155R71H104KE02J"
 			(at 133.35 77.47 0)
 			(effects
@@
 			)
 		)
-		(property "manf" "STMicroelectronics"
+		(property "Manufacturer" "STMicroelectronics"
 			(at 179.07 72.39 0)
 			(effects
@@
 			)
 		)
-		(property "manf#" "STM32G474RET3"
+		(property "Manufacturer Part Number" "STM32G474RET3"
 			(at 179.07 72.39 0)
 			(effects
@@
 			)
 		)
-		(property "manf" "KYOCERA AVX"
+		(property "Manufacturer" "KYOCERA AVX"
 			(at 133.35 118.11 0)
 			(effects
@@
 			)
 		)
-		(property "manf#" "CM05X5R475M25AH"
+		(property "Manufacturer Part Number" "CM05X5R475M25AH"
 			(at 133.35 118.11 0)
 			(effects
@@
 			)
 		)
-		(property "manf" "Würth Elektronik"
+		(property "Manufacturer" "Würth Elektronik"
 			(at 114.3 102.87 0)
 			(effects
@@
 			)
 		)
-		(property "manf#" "742792096"
+		(property "Manufacturer Part Number" "742792096"
 			(at 114.3 102.87 0)
 			(effects
@@
 			)
 		)
-		(property "manf" "Murata Electronics"
+		(property "Manufacturer" "Murata Electronics"
 			(at 133.35 99.06 0)
 			(effects
@@
 			)
 		)
-		(property "manf#" "GRM155Z71A105KE01J"
+		(property "Manufacturer Part Number" "GRM155Z71A105KE01J"
 			(at 133.35 99.06 0)
 			(effects
@@
 			)
 		)
-		(property "manf" "Murata Electronics"
+		(property "Manufacturer" "Murata Electronics"
 			(at 104.14 109.22 0)
 			(effects
@@
 			)
 		)
-		(property "manf#" "GRM155Z71A105KE01J"
+		(property "Manufacturer Part Number" "GRM155Z71A105KE01J"
 			(at 104.14 109.22 0)
 			(effects
@@
 			)
 		)
-		(property "manf" "Murata Electronics"
+		(property "Manufacturer" "Murata Electronics"
 			(at 148.59 55.88 0)
 			(effects
@@
 			)
 		)
-		(property "manf#" "GRM155Z71A105KE01J"
+		(property "Manufacturer Part Number" "GRM155Z71A105KE01J"
 			(at 148.59 55.88 0)
 			(effects
@@
 			)
 		)
-		(property "manf" "Murata Electronics"
+		(property "Manufacturer" "Murata Electronics"
 			(at 147.32 77.47 0)
 			(effects
@@
 			)
 		)
-		(property "manf#" "GCM155R71H104KE02J"
+		(property "Manufacturer Part Number" "GCM155R71H104KE02J"
 			(at 147.32 77.47 0)
 			(effects
@@
 			)
 		)
-		(property "manf" "Murata Electronics"
+		(property "Manufacturer" "Murata Electronics"
 			(at 149.86 118.11 0)
 			(effects
@@
 			)
 		)
-		(property "manf#" "GCM155R71H104KE02J"
+		(property "Manufacturer Part Number" "GCM155R71H104KE02J"
 			(at 149.86 118.11 0)
 			(effects
@@
 			)
 		)
-		(property "manf" "Murata Electronics"
+		(property "Manufacturer" "Murata Electronics"
 			(at 119.38 77.47 0)
 			(effects
@@
 			)
 		)
-		(property "manf#" "GCM155R71H104KE02J"
+		(property "Manufacturer Part Number" "GCM155R71H104KE02J"
 			(at 119.38 77.47 0)
 			(effects
@@
 			)
 		)
-		(property "manf" "Murata Electronics"
+		(property "Manufacturer" "Murata Electronics"
 			(at 88.9 77.47 0)
 			(effects
@@
 			)
 		)
-		(property "manf#" "GRM188Z71C475KE21J"
+		(property "Manufacturer Part Number" "GRM188Z71C475KE21J"
 			(at 88.9 77.47 0)
 			(effects
