File: Misc - Board Version DAC.kicad_sch (KiCad schematic)
At the start: 2 parts

Commit message: Updated files without navigate_results
Parts:
- R19, R20: Manufacturer (none) -> YAGEO; Manufacturer Part Number (none) -> RT0402FRE07100KL; manf YAGEO -> (none); manf# RT0402FRE07100KL -> (none)
Changed lines of the file:
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@@
 			)
 		)
-		(property "manf" "YAGEO"
+		(property "Manufacturer" "YAGEO"
 			(at 149.86 73.66 0)
 			(effects
@@
 			)
 		)
-		(property "manf#" "RT0402FRE07100KL"
+		(property "Manufacturer Part Number" "RT0402FRE07100KL"
 			(at 149.86 73.66 0)
 			(effects
@@
 			)
 		)
-		(property "manf" "YAGEO"
+		(property "Manufacturer" "YAGEO"
 			(at 149.86 55.88 0)
 			(effects
@@
 			)
 		)
-		(property "manf#" "RT0402FRE07100KL"
+		(property "Manufacturer Part Number" "RT0402FRE07100KL"
 			(at 149.86 55.88 0)
 			(effects
