File: Misc - Holes Fiducials.kicad_sch (KiCad schematic)
At the start: 15 parts

Commit message: Updated files without navigate_results
Parts:
- C130, C131, C132: Manufacturer (none) -> KEMET; Manufacturer Part Number (none) -> C0603V102KDRAC7867; manf KEMET -> (none); manf# C0603V102KDRAC7867 -> (none)
- R52, R53, R54: Manufacturer (none) -> Vishay; Manufacturer Part Number (none) -> CRCW06030000Z0EAHP; manf Vishay -> (none); manf# CRCW06030000Z0EAHP -> (none)
Changed lines of the file:
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@@
 			)
 		)
-		(property "manf" "KEMET"
+		(property "Manufacturer" "KEMET"
 			(at 82.55 91.44 0)
 			(effects
@@
 			)
 		)
-		(property "manf#" "C0603V102KDRAC7867"
+		(property "Manufacturer Part Number" "C0603V102KDRAC7867"
 			(at 82.55 91.44 0)
 			(effects
@@
 			)
 		)
-		(property "manf" "Vishay"
+		(property "Manufacturer" "Vishay"
 			(at 179.07 91.44 0)
 			(effects
@@
 			)
 		)
-		(property "manf#" "CRCW06030000Z0EAHP"
+		(property "Manufacturer Part Number" "CRCW06030000Z0EAHP"
 			(at 179.07 91.44 0)
 			(effects
@@
 			)
 		)
-		(property "manf" "KEMET"
+		(property "Manufacturer" "KEMET"
 			(at 162.56 91.44 0)
 			(effects
@@
 			)
 		)
-		(property "manf#" "C0603V102KDRAC7867"
+		(property "Manufacturer Part Number" "C0603V102KDRAC7867"
 			(at 162.56 91.44 0)
 			(effects
@@
 			)
 		)
-		(property "manf" "Vishay"
+		(property "Manufacturer" "Vishay"
 			(at 138.43 91.44 0)
 			(effects
@@
 			)
 		)
-		(property "manf#" "CRCW06030000Z0EAHP"
+		(property "Manufacturer Part Number" "CRCW06030000Z0EAHP"
 			(at 138.43 91.44 0)
 			(effects
@@
 			)
 		)
-		(property "manf" "Vishay"
+		(property "Manufacturer" "Vishay"
 			(at 99.06 91.44 0)
 			(effects
@@
 			)
 		)
-		(property "manf#" "CRCW06030000Z0EAHP"
+		(property "Manufacturer Part Number" "CRCW06030000Z0EAHP"
 			(at 99.06 91.44 0)
 			(effects
@@
 			)
 		)
-		(property "manf" "KEMET"
+		(property "Manufacturer" "KEMET"
 			(at 121.92 91.44 0)
 			(effects
@@
 			)
 		)
-		(property "manf#" "C0603V102KDRAC7867"
+		(property "Manufacturer Part Number" "C0603V102KDRAC7867"
 			(at 121.92 91.44 0)
 			(effects
