File: Motor Control - Inverter.kicad_sch (KiCad schematic)
At the start: 54 parts, among them J3 Phase A, J4 Phase B, J5 Phase C, Q1 TPW1R306PL,L1Q, Q2 TPW1R306PL,L1Q, Q3 TPW1R306PL,L1Q, Q4 TPW1R306PL,L1Q, Q5 TPW1R306PL,L1Q, Q6 TPW1R306PL,L1Q

Commit message: Updated files without navigate_results
Parts:
- C100, C96, C98: Manufacturer (none) -> Murata Electronics; Manufacturer Part Number (none) -> GRJ31CZ72A475KE01L; manf Murata Electronics -> (none); manf# GRJ31CZ72A475KE01L -> (none)
- C8: Manufacturer (none) -> Murata Electronics; Manufacturer Part Number (none) -> GRM155R72A332KA01D; manf Murata Electronics -> (none); manf# GRM155R72A332KA01D -> (none)
- C95, C97, C99: Manufacturer (none) -> KEMET; Manufacturer Part Number (none) -> C1206C104K1RACAUTO; manf KEMET -> (none); manf# C1206C104K1RACAUTO -> (none)
- D17: Manufacturer (none) -> STMicroelectronics; Manufacturer Part Number (none) -> BAT41KFILM; manf STMicroelectronics -> (none); manf# BAT41KFILM -> (none)
- Q1, Q2, Q3, Q4, Q5, Q6: Manufacturer (none) -> Toshiba Semiconductor and Storage; Manufacturer Part Number (none) -> TPW1R306PL,L1Q; manf Toshiba Semiconductor and Storage -> (none); manf# TPW1R306PL,L1Q -> (none)
- R10, R11, R13, R14, R16, R17: Manufacturer (none) -> Vishay; Manufacturer Part Number (none) -> CRCW08057R50FKEAHP; manf Vishay -> (none); manf# CRCW08057R50FKEAHP -> (none)
- R12, R15, R18: Manufacturer (none) -> Stackpole Electronics Inc; Manufacturer Part Number (none) -> HCS1206FTL500; manf Stackpole Electronics Inc -> (none); manf# HCS1206FTL500 -> (none)
- R23: Manufacturer (none) -> Stackpole Electronics Inc; Manufacturer Part Number (none) -> CSRT0603FT5R00; manf Stackpole Electronics Inc -> (none); manf# CSRT0603FT5R00 -> (none)
