File: Motor Control - Top Level.kicad_sch (KiCad schematic)
At the start: 25 parts, among them U6 DRV8353FS

Commit message: Updated files without navigate_results
Parts:
- C88, C93: Manufacturer (none) -> Taiyo Yuden; Manufacturer Part Number (none) -> TMK107AB7105KAHT; manf Taiyo Yuden -> (none); manf# TMK107AB7105KAHT -> (none)
- C89: Manufacturer (none) -> Murata Electronics; Manufacturer Part Number (none) -> GRJ31CZ72A475KE01L; manf Murata Electronics -> (none); manf# GRJ31CZ72A475KE01L -> (none)
- C90: Manufacturer (none) -> Murata Electronics; Manufacturer Part Number (none) -> GCM155R71C104KA55D; manf Murata Electronics -> (none); manf# GCM155R71C104KA55D -> (none)
- C91: Manufacturer (none) -> KEMET; Manufacturer Part Number (none) -> C0603C473K1RECAUTO; manf KEMET -> (none); manf# C0603C473K1RECAUTO -> (none)
- C92: Manufacturer (none) -> Taiyo Yuden; Manufacturer Part Number (none) -> HMK107B7104KAHT; manf Taiyo Yuden -> (none); manf# HMK107B7104KAHT -> (none)
- C94: Manufacturer (none) -> Murata Electronics; Manufacturer Part Number (none) -> GRT155R70J105KE01D; manf Murata Electronics -> (none); manf# GRT155R70J105KE01D -> (none)
- R8, R9: Manufacturer (none) -> Vishay; Manufacturer Part Number (none) -> ERJ-2RKF2001X; manf Vishay -> (none); manf# ERJ-2RKF2001X -> (none)
- U6: Manufacturer (none) -> Texas Instruments; Manufacturer Part Number (none) -> DRV8353FSRTAR; manf Texas Instruments -> (none); manf# DRV8353FSRTAR -> (none)
Changed lines of the file:
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@@
 			)
 		)
-		(property "manf" "Murata Electronics"
+		(property "Manufacturer" "Murata Electronics"
 			(at 110.49 156.21 0)
 			(effects
@@
 			)
 		)
-		(property "manf#" "GCM155R71C104KA55D"
+		(property "Manufacturer Part Number" "GCM155R71C104KA55D"
 			(at 110.49 156.21 0)
 			(effects
@@
 			)
 		)
-		(property "manf" "Taiyo Yuden"
+		(property "Manufacturer" "Taiyo Yuden"
 			(at 125.73 68.58 0)
 			(effects
@@
 			)
 		)
-		(property "manf#" "HMK107B7104KAHT"
+		(property "Manufacturer Part Number" "HMK107B7104KAHT"
 			(at 125.73 68.58 0)
 			(effects
@@
 			)
 		)
-		(property "manf" "Taiyo Yuden"
+		(property "Manufacturer" "Taiyo Yuden"
 			(at 125.73 104.14 0)
 			(effects
@@
 			)
 		)
-		(property "manf#" "TMK107AB7105KAHT"
+		(property "Manufacturer Part Number" "TMK107AB7105KAHT"
 			(at 125.73 104.14 0)
 			(effects
@@
 			)
 		)
-		(property "manf" "Murata Electronics"
+		(property "Manufacturer" "Murata Electronics"
 			(at 105.41 68.58 0)
 			(effects
@@
 			)
 		)
-		(property "manf#" "GRJ31CZ72A475KE01L"
+		(property "Manufacturer Part Number" "GRJ31CZ72A475KE01L"
 			(at 105.41 68.58 0)
 			(effects
@@
 			)
 		)
-		(property "manf" "Murata Electronics"
+		(property "Manufacturer" "Murata Electronics"
 			(at 173.99 91.44 0)
 			(effects
@@
 			)
 		)
-		(property "manf#" "GRT155R70J105KE01D"
+		(property "Manufacturer Part Number" "GRT155R70J105KE01D"
 			(at 173.99 91.44 0)
 			(effects
@@
 			)
 		)
-		(property "manf" "Vishay"
+		(property "Manufacturer" "Vishay"
 			(at 82.55 184.15 0)
 			(effects
@@
 			)
 		)
-		(property "manf#" "ERJ-2RKF2001X"
+		(property "Manufacturer Part Number" "ERJ-2RKF2001X"
 			(at 82.55 184.15 0)
 			(effects
@@
 			)
 		)
-		(property "manf" "Taiyo Yuden"
+		(property "Manufacturer" "Taiyo Yuden"
 			(at 85.09 73.66 0)
 			(effects
@@
 			)
 		)
-		(property "manf#" "TMK107AB7105KAHT"
+		(property "Manufacturer Part Number" "TMK107AB7105KAHT"
 			(at 85.09 73.66 0)
 			(effects
@@
 			)
 		)
-		(property "manf" "KEMET"
+		(property "Manufacturer" "KEMET"
 			(at 118.11 91.44 0)
 			(effects
@@
 			)
 		)
-		(property "manf#" "C0603C473K1RECAUTO"
+		(property "Manufacturer Part Number" "C0603C473K1RECAUTO"
 			(at 118.11 91.44 0)
 			(effects
@@
 			)
 		)
-		(property "manf" "Texas Instruments"
+		(property "Manufacturer" "Texas Instruments"
 			(at 151.13 170.18 0)
 			(effects
@@
 			)
 		)
-		(property "manf#" "DRV8353FSRTAR"
+		(property "Manufacturer Part Number" "DRV8353FSRTAR"
 			(at 151.13 170.18 0)
 			(effects
@@
 			)
 		)
-		(property "manf" "Vishay"
+		(property "Manufacturer" "Vishay"
 			(at 102.87 106.68 0)
 			(effects
@@
 			)
 		)
-		(property "manf#" "ERJ-2RKF2001X"
+		(property "Manufacturer Part Number" "ERJ-2RKF2001X"
 			(at 102.87 106.68 0)
 			(effects
