File: Power - Connectors.kicad_sch (KiCad schematic)
At the start: 4 parts, among them J1 XT60PW-F, J2 XT60PW-M

Commit message: Updated files without navigate_results
Parts:
- D1, D2: Manufacturer (none) -> Vishay; Manufacturer Part Number (none) -> SMBJ51CD-M3/H; manf Vishay -> (none); manf# SMBJ51CD-M3/H -> (none)
- J1: Manufacturer (none) -> AMASS; Manufacturer Part Number (none) -> XT60PW-F; manf AMASS -> (none); manf# XT60PW-F -> (none)
- J2: Manufacturer (none) -> AMASS; Manufacturer Part Number (none) -> XT60PW-M; manf AMASS -> (none); manf# XT60PW-M -> (none)
Changed lines of the file:
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@@
 			)
 		)
-		(property "manf" "AMASS"
+		(property "Manufacturer" "AMASS"
 			(at 115.57 90.17 0)
 			(effects
@@
 			)
 		)
-		(property "manf#" "XT60PW-M"
+		(property "Manufacturer Part Number" "XT60PW-M"
 			(at 115.57 90.17 0)
 			(effects
@@
 			)
 		)
-		(property "manf" "Vishay"
-			(at 149.86 77.47 0)
-			(effects
-				(font
-					(size 1.27 1.27)
-				)
-				(hide yes)
-			)
-		)
-		(property "manf#" "SMBJ51CD-M3/H"
+		(property "Manufacturer" "Vishay"
+			(at 149.86 77.47 0)
+			(effects
+				(font
+					(size 1.27 1.27)
+				)
+				(hide yes)
+			)
+		)
+		(property "Manufacturer Part Number" "SMBJ51CD-M3/H"
 			(at 149.86 77.47 0)
 			(effects
@@
 			)
 		)
-		(property "manf" "Vishay"
-			(at 172.72 77.47 0)
-			(effects
-				(font
-					(size 1.27 1.27)
-				)
-				(hide yes)
-			)
-		)
-		(property "manf#" "SMBJ51CD-M3/H"
+		(property "Manufacturer" "Vishay"
+			(at 172.72 77.47 0)
+			(effects
+				(font
+					(size 1.27 1.27)
+				)
+				(hide yes)
+			)
+		)
+		(property "Manufacturer Part Number" "SMBJ51CD-M3/H"
 			(at 172.72 77.47 0)
 			(effects
@@
 			)
 		)
-		(property "manf" "AMASS"
-			(at 115.57 67.31 0)
-			(effects
-				(font
-					(size 1.27 1.27)
-				)
-				(hide yes)
-			)
-		)
-		(property "manf#" "XT60PW-F"
-			(at 115.57 67.31 0)
-			(effects
+		(property "Manufacturer" "AMASS"
+			(at 115.57 67.31 0)
+			(effects
+				(font
+					(size 1.27 1.27)
+				)
+				(hide yes)
+			)
+		)
+		(property "Manufacturer Part Number" "XT60PW-F"
+			(at 115.57 67.31 0)
+			(effects
