File: Power - Generation.kicad_sch (KiCad schematic)
At the start: 110 parts, among them U2 LMR36506MSC5RPERQ1, U3 LMR36006FSCQ, U4 TPS62172DSG, U5 LP2992IM5-3.3/NOPB

Commit message: Updated files without navigate_results
Parts:
- C15, C16, C17, C18, C20, C45, C52: Manufacturer (none) -> TDK Corporation; Manufacturer Part Number (none) -> CGA4J1X7R2A225K125AC; manf TDK Corporation -> (none); manf# CGA4J1X7R2A225K125AC -> (none)
- C19, C21, C31, C32, C33, C34, C35, C36, C39, C40, C41, C42, C43, C44, C46, C47, C48, C49, C50, C51, C53, C54, C55, C57, C58, C59, C61, C62, C63, C64, C65, C66, C67, C68, C69, C70, C71, C72, C73, C74, C75, C77, C78, C79, C80, C81, C82, C85, C86, C87: Manufacturer (none) -> Murata Electronics; Manufacturer Part Number (none) -> GRJ31CZ72A475KE01L; manf Murata Electronics -> (none); manf# GRJ31CZ72A475KE01L -> (none)
- C22: Manufacturer (none) -> Taiyo Yuden; Manufacturer Part Number (none) -> HMK107B7104KAHT; manf Taiyo Yuden -> (none); manf# HMK107B7104KAHT -> (none)
- C23, C25: Manufacturer (none) -> Taiyo Yuden; Manufacturer Part Number (none) -> HMK107C7224KAHTE; manf Taiyo Yuden -> (none); manf# HMK107C7224KAHTE -> (none)
- C24, C26: Manufacturer (none) -> Murata Electronics; Manufacturer Part Number (none) -> GRM155Z71A105KE01J; manf Murata Electronics -> (none); manf# GRM155Z71A105KE01J -> (none)
- C27, C28, C29: Manufacturer (none) -> Murata Electronics; Manufacturer Part Number (none) -> GCM155R71H104KE02J; manf Murata Electronics -> (none); manf# GCM155R71H104KE02J -> (none)
- C30, C38: Manufacturer (none) -> TDK Corporation; Manufacturer Part Number (none) -> CGA6M3X7R1E156M200AB; manf TDK Corporation -> (none); manf# CGA6M3X7R1E156M200AB -> (none)
- C37, C83: Manufacturer (none) -> Murata Electronics; Manufacturer Part Number (none) -> GRM21BZ71A226ME15L; manf Murata Electronics -> (none); manf# GRM21BZ71A226ME15L -> (none)
- C56: Manufacturer (none) -> Murata Electronics; Manufacturer Part Number (none) -> GRM21BZ71E106KE15L; manf Murata Electronics -> (none); manf# GRM21BZ71E106KE15L -> (none)
- C60: Manufacturer (none) -> Taiyo Yuden; Manufacturer Part Number (none) -> TMK107AB7105KAHT; manf Taiyo Yuden -> (none); manf# TMK107AB7105KAHT -> (none)
- C76: Manufacturer (none) -> Taiyo Yuden; Manufacturer Part Number (none) -> HMR105B7103KV-F; manf Taiyo Yuden -> (none); manf# HMR105B7103KV-F -> (none)
- C84: Manufacturer (none) -> Murata Electronics; Manufacturer Part Number (none) -> GRM188Z71C475KE21J; manf Murata Electronics -> (none); manf# GRM188Z71C475KE21J -> (none)
- FB2, FB3, FB4: Manufacturer (none) -> Würth Elektronik; Manufacturer Part Number (none) -> 742792096; manf Würth Elektronik -> (none); manf# 742792096 -> (none)
- L1, L2: Manufacturer (none) -> Coilcraft; Manufacturer Part Number (none) -> LPS4018-223MRC; manf Coilcraft -> (none); manf# LPS4018-223MRC -> (none)
- L3: Manufacturer (none) -> Coilcraft; Manufacturer Part Number (none) -> LPS3314-222MRC; manf Coilcraft -> (none); manf# LPS3314-222MRC -> (none)
- R28: Manufacturer (none) -> YAGEO; Manufacturer Part Number (none) -> RT0402FRE0710KL; manf YAGEO -> (none); manf# RT0402FRE0710KL -> (none)
- R4: Manufacturer (none) -> Panasonic Electronic Components; Manufacturer Part Number (none) -> ERJ-2GE0R00X; manf Panasonic Electronic Components -> (none); manf# ERJ-2GE0R00X -> (none)
- R5: Manufacturer (none) -> YAGEO; Manufacturer Part Number (none) -> RT0402FRE07100KL; manf YAGEO -> (none); manf# RT0402FRE07100KL -> (none)
- R6: Manufacturer (none) -> YAGEO; Manufacturer Part Number (none) -> RT0402FRE079K09L; manf YAGEO -> (none); manf# RT0402FRE079K09L -> (none)
- U2: Manufacturer (none) -> Texas Instruments; Manufacturer Part Number (none) -> LMR36503MSC5RPERQ1; manf Texas Instruments -> (none); manf# LMR36503MSC5RPERQ1 -> (none)
- U3: Manufacturer (none) -> Texas Instruments; Manufacturer Part Number (none) -> LMR36006FSCQRNXTQ1; manf Texas Instruments -> (none); manf# LMR36006FSCQRNXTQ1 -> (none)
- U4: Manufacturer (none) -> Texas Instruments; Manufacturer Part Number (none) -> TPS62172DSGR; manf Texas Instruments -> (none); manf# TPS62172DSGR -> (none)
- U5: Manufacturer (none) -> Texas Instruments; Manufacturer Part Number (none) -> LP2992IM5-3.3/NOPB; manf Texas Instruments -> (none); manf# LP2992IM5-3.3/NOPB -> (none)
