File: Sensing - Battery.kicad_sch (KiCad schematic)
At the start: 3 parts

Commit message: Updated files without navigate_results
Parts:
- C103: Manufacturer (none) -> Murata Electronics; Manufacturer Part Number (none) -> GCM155R71H104KE02J; manf Murata Electronics -> (none); manf# GCM155R71H104KE02J -> (none)
- R29: Manufacturer (none) -> YAGEO; Manufacturer Part Number (none) -> RT0402FRE07100KL; manf YAGEO -> (none); manf# RT0402FRE07100KL -> (none)
- R30: Manufacturer (none) -> YAGEO; Manufacturer Part Number (none) -> RT0402FRE134K7L; manf YAGEO -> (none); manf# RT0402FRE134K7L -> (none)
Changed lines of the file:
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@@
 			)
 		)
-		(property "manf" "YAGEO"
+		(property "Manufacturer" "YAGEO"
 			(at 134.62 78.74 0)
 			(effects
@@
 			)
 		)
-		(property "manf#" "RT0402FRE134K7L"
+		(property "Manufacturer Part Number" "RT0402FRE134K7L"
 			(at 134.62 78.74 0)
 			(effects
@@
 			)
 		)
-		(property "manf" "Murata Electronics"
-			(at 151.13 78.74 0)
-			(effects
-				(font
-					(size 1.27 1.27)
-				)
-				(hide yes)
-			)
-		)
-		(property "manf#" "GCM155R71H104KE02J"
+		(property "Manufacturer" "Murata Electronics"
+			(at 151.13 78.74 0)
+			(effects
+				(font
+					(size 1.27 1.27)
+				)
+				(hide yes)
+			)
+		)
+		(property "Manufacturer Part Number" "GCM155R71H104KE02J"
 			(at 151.13 78.74 0)
 			(effects
@@
 			)
 		)
-		(property "manf" "YAGEO"
-			(at 134.62 63.5 0)
-			(effects
-				(font
-					(size 1.27 1.27)
-				)
-				(hide yes)
-			)
-		)
-		(property "manf#" "RT0402FRE07100KL"
-			(at 134.62 63.5 0)
-			(effects
+		(property "Manufacturer" "YAGEO"
+			(at 134.62 63.5 0)
+			(effects
+				(font
+					(size 1.27 1.27)
+				)
+				(hide yes)
+			)
+		)
+		(property "Manufacturer Part Number" "RT0402FRE07100KL"
+			(at 134.62 63.5 0)
+			(effects
