File: Sensing - Position.kicad_sch (KiCad schematic)
At the start: 7 parts, among them U7 AS5047P, U8 AS5048B

Commit message: Updated files without navigate_results
Parts:
- C104, C105: Manufacturer (none) -> Murata Electronics; Manufacturer Part Number (none) -> GCM155R71H104KE02J; manf Murata Electronics -> (none); manf# GCM155R71H104KE02J -> (none)
- C106: Manufacturer (none) -> Murata Electronics; Manufacturer Part Number (none) -> GRM21BZ71E106KE15L; manf Murata Electronics -> (none); manf# GRM21BZ71E106KE15L -> (none)
- R31, R32: Manufacturer (none) -> Panasonic Electronic Components; Manufacturer Part Number (none) -> ERJ-2GE0R00X; manf Panasonic Electronic Components -> (none); manf# ERJ-2GE0R00X -> (none)
- U7: Manufacturer (none) -> ams-OSRAM USA INC.; Manufacturer Part Number (none) -> AS5047P-ATSM; manf ams-OSRAM USA INC. -> (none); manf# AS5047P-ATSM -> (none)
- U8: Manufacturer (none) -> ams-OSRAM USA INC.; Manufacturer Part Number (none) -> AS5048B-HTSP-500; manf ams-OSRAM USA INC. -> (none); manf# AS5048B-HTSP-500 -> (none)
Changed lines of the file:
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@@
 			)
 		)
-		(property "manf" "Murata Electronics"
+		(property "Manufacturer" "Murata Electronics"
 			(at 50.8 92.71 0)
 			(effects
@@
 			)
 		)
-		(property "manf#" "GCM155R71H104KE02J"
+		(property "Manufacturer Part Number" "GCM155R71H104KE02J"
 			(at 50.8 92.71 0)
 			(effects
@@
 			)
 		)
-		(property "manf" "Panasonic Electronic Components"
+		(property "Manufacturer" "Panasonic Electronic Components"
 			(at 74.93 68.58 0)
 			(effects
@@
 			)
 		)
-		(property "manf#" "ERJ-2GE0R00X"
+		(property "Manufacturer Part Number" "ERJ-2GE0R00X"
 			(at 74.93 68.58 0)
 			(effects
@@
 			)
 		)
-		(property "manf" "Murata Electronics"
+		(property "Manufacturer" "Murata Electronics"
 			(at 220.98 74.93 0)
 			(effects
@@
 			)
 		)
-		(property "manf#" "GRM21BZ71E106KE15L"
+		(property "Manufacturer Part Number" "GRM21BZ71E106KE15L"
 			(at 220.98 74.93 0)
 			(effects
@@
 			)
 		)
-		(property "manf" "ams-OSRAM USA INC."
+		(property "Manufacturer" "ams-OSRAM USA INC."
 			(at 78.74 93.98 0)
 			(effects
@@
 			)
 		)
-		(property "manf#" "AS5047P-ATSM"
+		(property "Manufacturer Part Number" "AS5047P-ATSM"
 			(at 78.74 93.98 0)
 			(effects
@@
 			)
 		)
-		(property "manf" "ams-OSRAM USA INC."
+		(property "Manufacturer" "ams-OSRAM USA INC."
 			(at 204.47 93.98 0)
 			(effects
@@
 			)
 		)
-		(property "manf#" "AS5048B-HTSP-500"
+		(property "Manufacturer Part Number" "AS5048B-HTSP-500"
 			(at 204.47 93.98 0)
 			(effects
@@
 			)
 		)
-		(property "manf" "Panasonic Electronic Components"
+		(property "Manufacturer" "Panasonic Electronic Components"
 			(at 201.93 68.58 0)
 			(effects
@@
 			)
 		)
-		(property "manf#" "ERJ-2GE0R00X"
+		(property "Manufacturer Part Number" "ERJ-2GE0R00X"
 			(at 201.93 68.58 0)
 			(effects
@@
 			)
 		)
-		(property "manf" "Murata Electronics"
+		(property "Manufacturer" "Murata Electronics"
 			(at 175.26 92.71 0)
 			(effects
@@
 			)
 		)
-		(property "manf#" "GCM155R71H104KE02J"
+		(property "Manufacturer Part Number" "GCM155R71H104KE02J"
 			(at 175.26 92.71 0)
 			(effects
