File: Sensing - Temperature.kicad_sch (KiCad schematic)
At the start: 9 parts

Commit message: Updated files without navigate_results
Parts:
- C101, C102: Manufacturer (none) -> Murata Electronics; Manufacturer Part Number (none) -> GCM155R71H104KE02J; manf Murata Electronics -> (none); manf# GCM155R71H104KE02J -> (none)
- D17: Manufacturer (none) -> STMicroelectronics; Manufacturer Part Number (none) -> BAT41KFILM; manf STMicroelectronics -> (none); manf# BAT41KFILM -> (none)
- R27: Manufacturer (none) -> YAGEO; Manufacturer Part Number (none) -> RT0402FRE0710KL; manf YAGEO -> (none); manf# RT0402FRE0710KL -> (none)
- R44: Manufacturer (none) -> Vishay; Manufacturer Part Number (none) -> ERJ-2RKF2001X; manf Vishay -> (none); manf# ERJ-2RKF2001X -> (none)
- TH1: Manufacturer (none) -> Murata Electronics; Manufacturer Part Number (none) -> NCP15WB473F03RC; manf Murata Electronics -> (none); manf# NCP15WB473F03RC -> (none)
Changed lines of the file:
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@@
 			)
 		)
-		(property "manf" "YAGEO"
+		(property "Manufacturer" "YAGEO"
 			(at 97.79 101.6 0)
 			(effects
@@
 			)
 		)
-		(property "manf#" "RT0402FRE0710KL"
+		(property "Manufacturer Part Number" "RT0402FRE0710KL"
 			(at 97.79 101.6 0)
 			(effects
@@
 			)
 		)
-		(property "manf" "Vishay"
+		(property "Manufacturer" "Vishay"
 			(at 176.53 101.6 0)
 			(effects
@@
 			)
 		)
-		(property "manf#" "ERJ-2RKF2001X"
+		(property "Manufacturer Part Number" "ERJ-2RKF2001X"
 			(at 176.53 101.6 0)
 			(effects
@@
 			)
 		)
-		(property "manf" "Murata Electronics"
+		(property "Manufacturer" "Murata Electronics"
 			(at 111.76 101.6 0)
 			(effects
@@
 			)
 		)
-		(property "manf#" "GCM155R71H104KE02J"
+		(property "Manufacturer Part Number" "GCM155R71H104KE02J"
 			(at 111.76 101.6 0)
 			(effects
@@
 			)
 		)
-		(property "manf" "STMicroelectronics"
+		(property "Manufacturer" "STMicroelectronics"
 			(at 194.31 87.63 0)
 			(effects
@@
 			)
 		)
-		(property "manf#" "BAT41KFILM"
+		(property "Manufacturer Part Number" "BAT41KFILM"
 			(at 194.31 87.63 0)
 			(effects
@@
 			)
 		)
-		(property "manf" "STMicroelectronics"
+		(property "Manufacturer" "STMicroelectronics"
 			(at 120.65 85.09 0)
 			(effects
@@
 			)
 		)
-		(property "manf#" "BAT41KFILM"
+		(property "Manufacturer Part Number" "BAT41KFILM"
 			(at 120.65 85.09 0)
 			(effects
@@
 			)
 		)
-		(property "manf" "Murata Electronics"
+		(property "Manufacturer" "Murata Electronics"
 			(at 97.79 82.55 0)
 			(effects
@@
 			)
 		)
-		(property "manf#" "NCP15WB473F03RC"
+		(property "Manufacturer Part Number" "NCP15WB473F03RC"
 			(at 97.79 82.55 0)
 			(effects
@@
 			)
 		)
-		(property "manf" "Murata Electronics"
+		(property "Manufacturer" "Murata Electronics"
 			(at 190.5 101.6 0)
 			(effects
@@
 			)
 		)
-		(property "manf#" "GCM155R71H104KE02J"
+		(property "Manufacturer Part Number" "GCM155R71H104KE02J"
 			(at 190.5 101.6 0)
 			(effects
