File: User - LED Indicators.kicad_sch (KiCad schematic)
At the start: 10 parts, among them Q7 PMV90ENER, Q8 PMV90ENER

Commit message: Updated files without navigate_results
Parts:
- D12: Manufacturer (none) -> Bivar Inc.; Manufacturer Part Number (none) -> SM1206NYC-IL; manf Bivar Inc. -> (none); manf# SM1206NYC-IL -> (none)
- D13: Manufacturer (none) -> Bivar Inc.; Manufacturer Part Number (none) -> SM1206NPGC-IL; manf Bivar Inc. -> (none); manf# SM1206NPGC-IL -> (none)
- Q7, Q8: Manufacturer (none) -> Nexperia USA Inc.; Manufacturer Part Number (none) -> PMV90ENER; manf Nexperia USA Inc. -> (none); manf# PMV90ENER -> (none)
- R18: Manufacturer (none) -> YAGEO; Manufacturer Part Number (none) -> RT0402FRE07100KL; manf YAGEO -> (none); manf# RT0402FRE07100KL -> (none)
- R22, R23, R25: Manufacturer (none) -> Vishay; Manufacturer Part Number (none) -> RCS0402100RFKED; manf Vishay -> (none); manf# RCS0402100RFKED -> (none)
- R26: Manufacturer (none) -> Vishay; Manufacturer Part Number (none) -> RCS0402150RFKED; manf Vishay -> (none); manf# RCS0402150RFKED -> (none)
Changed lines of the file:
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@@
 			)
 		)
-		(property "manf" "Nexperia USA Inc."
+		(property "Manufacturer" "Nexperia USA Inc."
 			(at 147.32 96.52 0)
 			(effects
@@
 			)
 		)
-		(property "manf#" "PMV90ENER"
+		(property "Manufacturer Part Number" "PMV90ENER"
 			(at 147.32 96.52 0)
 			(effects
@@
 			)
 		)
-		(property "manf" "Vishay"
+		(property "Manufacturer" "Vishay"
 			(at 134.62 96.52 0)
 			(effects
@@
 			)
 		)
-		(property "manf#" "RCS0402100RFKED"
+		(property "Manufacturer Part Number" "RCS0402100RFKED"
 			(at 134.62 96.52 0)
 			(effects
@@
 			)
 		)
-		(property "manf" "Nexperia USA Inc."
+		(property "Manufacturer" "Nexperia USA Inc."
 			(at 195.58 96.52 0)
 			(effects
@@
 			)
 		)
-		(property "manf#" "PMV90ENER"
+		(property "Manufacturer Part Number" "PMV90ENER"
 			(at 195.58 96.52 0)
 			(effects
@@
 			)
 		)
-		(property "manf" "Vishay"
+		(property "Manufacturer" "Vishay"
 			(at 198.12 67.31 0)
 			(effects
@@
 			)
 		)
-		(property "manf#" "RCS0402150RFKED"
+		(property "Manufacturer Part Number" "RCS0402150RFKED"
 			(at 198.12 67.31 0)
 			(effects
@@
 			)
 		)
-		(property "manf" "YAGEO"
+		(property "Manufacturer" "YAGEO"
 			(at 128.27 102.87 0)
 			(effects
@@
 			)
 		)
-		(property "manf#" "RT0402FRE07100KL"
+		(property "Manufacturer Part Number" "RT0402FRE07100KL"
 			(at 128.27 102.87 0)
 			(effects
@@
 			)
 		)
-		(property "manf" "Bivar Inc."
+		(property "Manufacturer" "Bivar Inc."
 			(at 198.12 81.28 0)
 			(effects
@@
 			)
 		)
-		(property "manf#" "SM1206NPGC-IL"
+		(property "Manufacturer Part Number" "SM1206NPGC-IL"
 			(at 198.12 81.28 0)
 			(effects
@@
 			)
 		)
-		(property "manf" "Vishay"
+		(property "Manufacturer" "Vishay"
 			(at 182.88 96.52 0)
 			(effects
@@
 			)
 		)
-		(property "manf#" "RCS0402100RFKED"
+		(property "Manufacturer Part Number" "RCS0402100RFKED"
 			(at 182.88 96.52 0)
 			(effects
@@
 			)
 		)
-		(property "manf" "YAGEO"
+		(property "Manufacturer" "YAGEO"
 			(at 176.53 102.87 0)
 			(effects
@@
 			)
 		)
-		(property "manf#" "RT0402FRE07100KL"
+		(property "Manufacturer Part Number" "RT0402FRE07100KL"
 			(at 176.53 102.87 0)
 			(effects
@@
 			)
 		)
-		(property "manf" "Bivar Inc."
+		(property "Manufacturer" "Bivar Inc."
 			(at 149.86 81.28 0)
 			(effects
@@
 			)
 		)
-		(property "manf#" "SM1206NYC-IL"
+		(property "Manufacturer Part Number" "SM1206NYC-IL"
 			(at 149.86 81.28 0)
 			(effects
@@
 			)
 		)
-		(property "manf" "Vishay"
+		(property "Manufacturer" "Vishay"
 			(at 149.86 67.31 0)
 			(effects
@@
 			)
 		)
-		(property "manf#" "RCS0402100RFKED"
+		(property "Manufacturer Part Number" "RCS0402100RFKED"
 			(at 149.86 67.31 0)
 			(effects
